Commit message: control joint from python

File: gz/models/rrbot/rrbot.sdf.xacro (robot description, xacro)
@@ -38,4 +38,7 @@
             <axis>
                 <xyz>1 0 0</xyz>
+                <dynamics>
+                    <damping>0.5</damping>
+                  </dynamics>
             </axis>
         </joint>
@@ -53,4 +56,7 @@
             <axis>
                 <xyz>1 0 0</xyz>
+                <dynamics>
+                    <damping>0.5</damping>
+                  </dynamics>
             </axis>
         </joint>
@@ -78,4 +84,5 @@
             <xacro:camera name="camera1" rate="20" width="640" height="480" fov="50"/>
         </link>
+        <plugin name="joint_control" filename="libJointForcePlugin.so"/>
     </model>
 </sdf>
